File: testPCB/testPCB.kicad_pcb (KiCad board)
At the start: 2 copper layers, 8 parts, among them U1 AP2112K-3.3, U2 LSM6DSV

Commit message: Testing Changes
Verifying library functionalities
Parts:
- added J1: USB4125-GF-A, Rover:CONN6_USB4125_GCT, F.Cu at (47.9, 30.0)
- added U3: LSM6DSV, Rover:LSM6DSV, F.Cu at (43.8, 36.1)
Other:
- board outline added: 8.7 x 4.4 mm
