File: single_board/single_board/single_board.kicad_sch (KiCad schematic)
At the start: 81 parts, among them J1 5V, J10 PWM2, J11 PWM3, J12 PWM4, J13 PWM45, J14 PWM6, J15 BOOTSEL, J16 SWD, J17 UART, J18 CAN_OUT, J19 SPI Debug, J2 v3v3, J3 ENC1, J4 ENC2, J5 ENC3, J6 ENC4, J7 ENC5, J8 ENC6, J9 PWM1, SW1 Button, U1 USBLC6-2SC6, U2 AP2112K-3.3, U3 STM32G474VBTx, U4 TJA1042T-3, U5 LSM6DSVTR, Y1 FC-135

Commit message: Clean up copied schematic
Parts:
- R5, R6: value 62 -> 60
Other:
- note added: "Data line resistors & Current limiting resistors"
- note removed: "Board critical 5V ESD Protection"
- note removed: "Consider 52 ohm with 68 ohm. 120 ohm series resistance. Creates two low pass filters with different cutoff frequencies."
- note removed: "Data line resistors & Current limitin resistors"
- note removed: "Ground standby; less features to configure. Assuming power saving is minimal"
- note removed: "Look into common ground/shielding for CAN bus"
Changed lines of the file:
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@@
 	(generator_version "10.0")
 	(paper "A3")
-	(text "Board critical 5V ESD Protection"
-		(exclude_from_sim no)
-		(at 82.55 47.752 0)
-		(effects
-			(font
-				(size 1.27 1.27)
-			)
-		)
-	)
 	(text "Mode 1\nSPI 4-wire"
 		(exclude_from_sim no)
@@
 	(text "AH1014\nSplit termination resistor values\nC_split 4.7nf-10nf"
 		(exclude_from_sim no)
-		(at 258.064 69.342 0)
+		(at 261.366 63.5 0)
 		(effects
 			(font
@@
 		)
 	)
-	(text "Look into common ground/shielding for CAN bus"
+	(text "Data line resistors &\nCurrent limiting resistors"
 		(exclude_from_sim no)
-		(at 306.07 60.198 0)
-		(effects
-			(font
-				(size 1.27 1.27)
-			)
-		)
-	)
-	(text "Data line resistors &\nCurrent limitin resistors"
-		(exclude_from_sim no)
-		(at 388.366 61.214 0)
+		(at 371.602 61.214 0)
 		(effects
 			(font
@@
 		)
 	)
-	(text "Ground standby; less features to configure.\nAssuming power saving is minimal"
-		(exclude_from_sim no)
-		(at 199.136 60.96 0)
-		(effects
-			(font
-				(size 1.27 1.27)
-			)
-			(justify left)
-		)
-	)
 	(text "Extra 1uf decoupling"
 		(exclude_from_sim no)
@@
 		)
 	)
-	(text "Consider 52 ohm with 68 ohm. \n120 ohm series resistance.\nCreates two low pass filters with different cutoff frequencies.\n"
-		(exclude_from_sim no)
-		(at 258.318 82.296 0)
-		(effects
-			(font
-				(size 1.27 1.27)
-			)
-			(justify left)
-		)
-	)
 	(text "CAN Transciever"
 		(exclude_from_sim no)
@@
 			)
 		)
-		(property "Value" "62"
+		(property "Value" "60"
 			(at 276.86 38.0999 0)
 			(show_name no)
@@
 			)
 		)
-		(property "Value" "62"
+		(property "Value" "60"
 			(at 276.86 50.7999 0)
 			(show_name no)
